File: MXBreakout.kicad_pcb (KiCad board)
At the start: 2 copper layers, 27.9 x 19 mm, 16 parts, among them U1 Wii-MX, X1 32.768kHz

Commit message: initial changes
Parts:
- removed TP4: DATA0, TestPoint:TestPoint_Pad_D1.0mm
- removed TP5: DATA1, TestPoint:TestPoint_Pad_D1.0mm
- removed TP6: DATA2, TestPoint:TestPoint_Pad_D1.0mm
- removed TP7: DATA3, TestPoint:TestPoint_Pad_D1.0mm
Connections:
- U1 pad 11: Net-(U1-DATA0) -> /DATA0
- U1 pad 12: Net-(U1-DATA1) -> /DATA1
- U1 pad 13: Net-(U1-DATA2) -> /DATA2
- U1 pad 14: Net-(U1-DATA3) -> /DATA3
Routing:
- net /DATA2: track 0.00 -> 2.37 mm, vias 0 -> 1
- net /DATA1: track 0.00 -> 2.37 mm, vias 0 -> 1
- net /DATA0: track 0.00 -> 2.36 mm, vias 0 -> 1
- net Net-(U1-DATA0): track 2.34 -> 0.00 mm
- net Net-(U1-DATA1): track 2.34 -> 0.00 mm
- net Net-(U1-DATA2): track 2.33 -> 0.00 mm
- net Net-(U1-DATA3): track 2.33 -> 0.00 mm
- net /DATA3: track 0.00 -> 2.33 mm, vias 0 -> 1
Changed lines of the file:
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@@
   (net 5 "Net-(D1-A)")
   (net 6 "Net-(R1-Pad2)")
-  (net 7 "Net-(U1-DATA0)")
-  (net 8 "Net-(U1-DATA1)")
-  (net 9 "Net-(U1-DATA2)")
-  (net 10 "Net-(U1-DATA3)")
+  (net 7 "/DATA0")
+  (net 8 "/DATA1")
+  (net 9 "/DATA2")
+  (net 10 "/DATA3")
   (net 11 "+3.3V")
   (net 12 "unconnected-(U1-U22-Pad20)")
@@
     (pad "10" smd roundrect (at -4.65 3.175) (size 2.05 0.6) (layers "F.Cu" "F.Paste" "F.Mask") (roundrect_rratio 0.25))
     (pad "11" smd roundrect (at -4.65 4.445) (size 2.05 0.6) (layers "F.Cu" "F.Paste" "F.Mask") (roundrect_rratio 0.25)
-      (net 7 "Net-(U1-DATA0)") (pinfunction "DATA0") (pintype "passive"))
+      (net 7 "/DATA0") (pinfunction "DATA0") (pintype "passive"))
     (pad "12" smd roundrect (at -4.65 5.715) (size 2.05 0.6) (layers "F.Cu" "F.Paste" "F.Mask") (roundrect_rratio 0.25)
-      (net 8 "Net-(U1-DATA1)") (pinfunction "DATA1") (pintype "passive"))
+      (net 8 "/DATA1") (pinfunction "DATA1") (pintype "passive"))
     (pad "13" smd roundrect (at -4.65 6.985) (size 2.05 0.6) (layers "F.Cu" "F.Paste" "F.Mask") (roundrect_rratio 0.25)
-      (net 9 "Net-(U1-DATA2)") (pinfunction "DATA2") (pintype "passive"))
+      (net 9 "/DATA2") (pinfunction "DATA2") (pintype "passive"))
     (pad "14" smd roundrect (at -4.65 8.255) (size 2.05 0.6) (layers "F.Cu" "F.Paste" "F.Mask") (roundrect_rratio 0.25)
-      (net 10 "Net-(U1-DATA3)") (pinfunction "DATA3") (pintype "passive"))
+      (net 10 "/DATA3") (pinfunction "DATA3") (pintype "passive"))
     (pad "15" smd roundrect (at 4.65 8.255) (size 2.05 0.6) (layers "F.Cu" "F.Paste" "F.Mask") (roundrect_rratio 0.25))
     (pad "16" smd roundrect (at 4.65 6.985) (size 2.05 0.6) (layers "F.Cu" "F.Paste" "F.Mask") (roundrect_rratio 0.25)
@@
   )
   (footprint "TestPoint:TestPoint_Pad_D1.0mm" (layer "F.Cu")
-    (at 116.2 93.5)
-    (descr "SMD pad as test Point, diameter 1.0mm")
-    (tags "test point SMD pad")
-    (property "Sheetfile" "MXBreakout.kicad_sch")
-    (property "Sheetname" "")
-    (property "ki_description" "test point")
-    (property "ki_keywords" "test point tp")
-    (attr exclude_from_pos_files)
-    (fp_text reference "TP4" (at 0 -1.448) (layer "F.Fab")
-        (effects (font (size 1 1) (thickness 0.15)))
-    )
-    (fp_text value "DATA0" (at 0 1.55) (layer "F.Fab")
-        (effects (font (size 1 1) (thickness 0.15)))
-    )
-    (fp_text user "${REFERENCE}" (at 0 -1.45) (layer "F.Fab")
-        (effects (font (size 1 1) (thickness 0.15)))
-    )
-    (fp_circle (center 0 0) (end 0 0.4)
-      (stroke (width 0.12) (type solid)) (fill none) (layer "F.SilkS"))
-    (fp_circle (center 0 0) (end 0.6 0)
-      (stroke (width 0.05) (type solid)) (fill none) (layer "F.CrtYd"))
-    (pad "1" smd circle (at 0 0) (size 0.75 0.75) (layers "F.Cu" "F.Mask")
-      (net 7 "Net-(U1-DATA0)") (pinfunction "1") (pintype "passive"))
-  )
-  (footprint "TestPoint:TestPoint_Pad_D1.0mm" (layer "F.Cu")
     (at 135.525 95.175)
     (descr "SMD pad as test Point, diameter 1.0mm")
@@
       (net 6 "Net-(R1-Pad2)") (pinfunction "1") (pintype "passive"))
   )
-  (footprint "TestPoint:TestPoint_Pad_D1.0mm" (layer "F.Cu")
-    (at 116.2 97.325)
-    (descr "SMD pad as test Point, diameter 1.0mm")
-    (tags "test point SMD pad")
-    (property "Sheetfile" "MXBreakout.kicad_sch")
-    (property "Sheetname" "")
-    (property "ki_description" "test point")
-    (property "ki_keywords" "test point tp")
-    (attr exclude_from_pos_files)
-    (fp_text reference "TP7" (at 0 -1.448) (layer "F.Fab")
-        (effects (font (size 1 1) (thickness 0.15)))
-    )
-    (fp_text value "DATA3" (at 0 1.55) (layer "F.Fab")
-        (effects (font (size 1 1) (thickness 0.15)))
-    )
-    (fp_text user "${REFERENCE}" (at 0 -1.45) (layer "F.Fab")
-        (effects (font (size 1 1) (thickness 0.15)))
-    )
-    (fp_circle (center 0 0) (end 0 0.4)
-      (stroke (width 0.12) (type solid)) (fill none) (layer "F.SilkS"))
-    (fp_circle (center 0 0) (end 0.6 0)
-      (stroke (width 0.05) (type solid)) (fill none) (layer "F.CrtYd"))
-    (pad "1" smd circle (at 0 0) (size 0.75 0.75) (layers "F.Cu" "F.Mask")
-      (net 10 "Net-(U1-DATA3)") (pinfunction "1") (pintype "passive"))
-  )
   (footprint "Capacitor_SMD:C_0402_1005Metric" (layer "F.Cu")
     (at 129.8 81.6 -90)
@@
       (rotate (xyz 0 0 0))
     )
-  )
-  (footprint "TestPoint:TestPoint_Pad_D1.0mm" (layer "F.Cu")
-    (at 116.2 96.05)
-    (descr "SMD pad as test Point, diameter 1.0mm")
-    (tags "test point SMD pad")
-    (property "Sheetfile" "MXBreakout.kicad_sch")
-    (property "Sheetname" "")
-    (property "ki_description" "test point")
-    (property "ki_keywords" "test point tp")
-    (attr exclude_from_pos_files)
-    (fp_text reference "TP6" (at 0 -1.448) (layer "F.Fab")
-        (effects (font (size 1 1) (thickness 0.15)))
-    )
-    (fp_text value "DATA2" (at 0 1.55) (layer "F.Fab")
-        (effects (font (size 1 1) (thickness 0.15)))
-    )
-    (fp_text user "${REFERENCE}" (at 0 -1.45) (layer "F.Fab")
-        (effects (font (size 1 1) (thickness 0.15)))
-    )
-    (fp_circle (center 0 0) (end 0 0.4)
-      (stroke (width 0.12) (type solid)) (fill none) (layer "F.SilkS"))
-    (fp_circle (center 0 0) (end 0.6 0)
-      (stroke (width 0.05) (type solid)) (fill none) (layer "F.CrtYd"))
-    (pad "1" smd circle (at 0 0) (size 0.75 0.75) (layers "F.Cu" "F.Mask")
-      (net 9 "Net-(U1-DATA2)") (pinfunction "1") (pintype "passive"))
-  )
-  (footprint "TestPoint:TestPoint_Pad_D1.0mm" (layer "F.Cu")
-    (at 116.2 94.775)
-    (descr "SMD pad as test Point, diameter 1.0mm")
-    (tags "test point SMD pad")
-    (property "Sheetfile" "MXBreakout.kicad_sch")
-    (property "Sheetname" "")
-    (property "ki_description" "test point")
-    (property "ki_keywords" "test point tp")
-    (attr exclude_from_pos_files)
-    (fp_text reference "TP5" (at 0 -1.448) (layer "F.Fab")
-        (effects (font (size 1 1) (thickness 0.15)))
-    )
-    (fp_text value "DATA1" (at 0 1.55) (layer "F.Fab")
-        (effects (font (size 1 1) (thickness 0.15)))
-    )
-    (fp_text user "${REFERENCE}" (at 0 -1.45) (layer "F.Fab")
-        (effects (font (size 1 1) (thickness 0.15)))
-    )
-    (fp_circle (center 0 0) (end 0 0.4)
-      (stroke (width 0.12) (type solid)) (fill none) (layer "F.SilkS"))
-    (fp_circle (center 0 0) (end 0.6 0)
-      (stroke (width 0.05) (type solid)) (fill none) (layer "F.CrtYd"))
-    (pad "1" smd circle (at 0 0) (size 0.75 0.75) (layers "F.Cu" "F.Mask")
-      (net 8 "Net-(U1-DATA1)") (pinfunction "1") (pintype "passive"))
   )
   (footprint "Capacitor_SMD:C_0402_1005Metric" (layer "F.Cu")
@@
   (segment (start 140.3 93.7) (end 140.3 88.85) (width 0.25) (layer "F.Cu") (net 6))
   (via (at 140.3 88.85) (size 1) (drill 0.5) (layers "F.Cu" "B.Cu") (net 6))
-  (segment (start 118.55 93.495) (end 116.205 93.495) (width 0.25) (layer "F.Cu") (net 7))
-  (segment (start 118.55 94.765) (end 116.21 94.765) (width 0.25) (layer "F.Cu") (net 8))
-  (segment (start 118.55 96.035) (end 116.215 96.035) (width 0.25) (layer "F.Cu") (net 9))
+  (segment (start 116.2 93.5) (end 116.205 93.495) (width 0.25) (layer "F.Cu") (net 7))
+  (segment (start 118.55 93.495) (end 116.2 93.5) (width 0.25) (layer "F.Cu") (net 7))
+  (via (at 116.2 93.5) (size 1) (drill 0.5) (layers "F.Cu" "B.Cu") (net 7))
+  (segment (start 116.2 94.75) (end 116.21 94.765) (width 0.25) (layer "F.Cu") (net 8))
+  (segment (start 118.55 94.765) (end 116.2 94.75) (width 0.25) (layer "F.Cu") (net 8))
+  (via (at 116.2 94.75) (size 1) (drill 0.5) (layers "F.Cu" "B.Cu") (net 8))
+  (segment (start 118.55 96.035) (end 116.2 96.05) (width 0.25) (layer "F.Cu") (net 9))
+  (segment (start 116.2 96.05) (end 116.215 96.035) (width 0.25) (layer "F.Cu") (net 9))
+  (via (at 116.2 96.05) (size 1) (drill 0.5) (layers "F.Cu" "B.Cu") (net 9))
   (segment (start 118.55 97.305) (end 116.22 97.305) (width 0.25) (layer "F.Cu") (net 10))
+  (via (at 116.2 97.3) (size 1) (drill 0.5) (layers "F.Cu" "B.Cu") (net 10))
   (segment (start 127.85 85.25) (end 127.85 85.875) (width 0.25) (layer "F.Cu") (net 11))
   (segment (start 126.825001 94.765) (end 126.5 94.439999) (width 0.25) (layer "F.Cu") (net 11))

Commit message: nearing completion
Parts:
- removed TP1: BATT, TestPoint:TestPoint_Pad_D4.0mm
- removed TP9: 3.3V, TestPoint:TestPoint_Pad_D1.0mm
- added TP10: TestPoint_2Pole, Resistor_SMD:R_0402_1005Metric, F.Cu at (132.0, 86.3)
- added TP11: U10, Wii:TestPoint_THTPad_D0.5mm_Drill0.35mm, F.Cu at (124.0, 84.0)
- added TP3: GND, Wii:TestPoint_THTPad_D0.5mm_Drill0.35mm, F.Cu at (135.6, 83.6)
- added TP4: TestPoint, Wii:TestPoint_THTPad_D0.5mm_Drill0.35mm, F.Cu at (124.0, 85.0)
- added TP5: TestPoint, Wii:TestPoint_THTPad_D0.5mm_Drill0.35mm, F.Cu at (129.5, 85.0)
- added TP6: TestPoint, Wii:TestPoint_THTPad_D0.5mm_Drill0.35mm, F.Cu at (128.8, 85.0)
- added TP7: TestPoint, Wii:TestPoint_THTPad_D0.5mm_Drill0.35mm, F.Cu at (123.0, 86.0)
- added U10: ~, Package_TO_SOT_SMD:SOT-23-5, F.Cu at (123.9, 89.1)
- TP2: footprint TestPoint:TestPoint_Pad_D4.0mm -> TestPoint:TestPoint_Pad_D1.0mm; moved to F.Cu
- TP3: footprint TestPoint:TestPoint_Pad_D1.0mm -> Wii:TestPoint_THTPad_D0.5mm_Drill0.35mm
- moved TP8 44.6 mm to (96.2, 100.9)
- moved D1 44.3 mm to (97.5, 95.5)
- moved R1 44.3 mm to (97.5, 98.0)
- moved C2 33.2 mm to (101.2, 97.9), turned to 90 degrees
- moved X1 30.7 mm to (104.8, 97.9), turned to 0 degrees
- moved C1 28.8 mm to (108.4, 97.9), turned to 90 degrees
- moved TP2 21.1 mm to (100.3, 100.9), turned to 0 degrees
- moved TP3 11.8 mm to (134.1, 83.6)
- moved U1 10.5 mm to (113.8, 84.2), turned to 180 degrees
- moved C3 2.71 mm to (131.5, 83.7), turned to 0 degrees
Routing:
- net +3.3V: track 30.0 -> 44.9 mm
- net /DATA2: track 2.37 -> 16.9 mm, vias 1 -> 0
- net /DATA3: track 2.33 -> 15.1 mm, vias 1 -> 0
- net /DATA1: track 2.37 -> 13.7 mm, vias 1 -> 0
- net Net-(U1-X_2): track 6.71 -> 16.5 mm
- net Net-(U1-X_1): track 6.69 -> 14.0 mm
- net /DATA0: track 2.36 -> 8.13 mm, vias 1 -> 0
- net Net-(U10-RST): track 0.00 -> 4.34 mm
- net Net-(R1-Pad2): track 6.55 -> 2.92 mm, vias 1 -> 0
- net Net-(D1-K): track 12.5 -> 14.6 mm, vias 0 -> 2
- net GND: vias 37 -> 24
Other:
- board size 27.9 x 19 mm -> 42.3 x 28.3 mm

Commit message: Updates
Parts:
- added REF**: TestPoint_THTPad_D0.5mm_Drill0.35mm, Wii:TestPoint_THTPad_D0.5mm_Drill0.35mm, F.Cu at (95.0, 102.5)
- added REF**: TestPoint_THTPad_D0.5mm_Drill0.35mm, Wii:TestPoint_THTPad_D0.5mm_Drill0.35mm, F.Cu at (90.0, 95.0)
- added REF**: TestPoint_THTPad_D0.5mm_Drill0.35mm, Wii:TestPoint_THTPad_D0.5mm_Drill0.35mm, F.Cu at (90.0, 98.8)
- added REF**: TestPoint_THTPad_D0.5mm_Drill0.35mm, Wii:TestPoint_THTPad_D0.5mm_Drill0.35mm, F.Cu at (90.0, 97.5)
- added REF**: TestPoint_THTPad_D0.5mm_Drill0.35mm, Wii:TestPoint_THTPad_D0.5mm_Drill0.35mm, F.Cu at (90.0, 96.2)
- added REF**: TestPoint_THTPad_D0.5mm_Drill0.35mm, Wii:TestPoint_THTPad_D0.5mm_Drill0.35mm, F.Cu at (92.5, 102.5)
- added REF**: TestPoint_THTPad_D0.5mm_Drill0.35mm, Wii:TestPoint_THTPad_D0.5mm_Drill0.35mm, F.Cu at (93.8, 102.5)
- added REF**: TestPoint_THTPad_D0.5mm_Drill0.35mm, Wii:TestPoint_THTPad_D0.5mm_Drill0.35mm, F.Cu at (103.8, 102.5)
- added REF**: TestPoint_THTPad_D0.5mm_Drill0.35mm, Wii:TestPoint_THTPad_D0.5mm_Drill0.35mm, F.Cu at (90.0, 100.0)
- added REF**: TestPoint_THTPad_D0.5mm_Drill0.35mm, Wii:TestPoint_THTPad_D0.5mm_Drill0.35mm, F.Cu at (102.5, 102.5)
- moved U10 8.44 mm to (122.9, 80.8), turned to -45 degrees
- moved TP2 4.93 mm to (95.3, 100.9)
- moved C1 4.93 mm to (103.5, 97.9)
- moved C2 4.93 mm to (96.3, 97.9)
- moved D1 4.93 mm to (92.6, 95.5)
- moved R1 4.93 mm to (92.6, 98.0)
- moved TP8 4.93 mm to (91.3, 100.9)
- moved X1 4.93 mm to (99.9, 97.9)
Routing:
- net +3.3V: track 44.9 -> 51.8 mm
- net Net-(D1-K): track 14.6 -> 19.3 mm
- net GND: track 0.00 -> 4.49 mm, vias 24 -> 30
- net Net-(U10-RST): track 4.34 -> 2.16 mm
- net /DATA2: track 16.9 -> 15.1 mm, vias 0 -> 1
- net Net-(U1-X_2): track 16.5 -> 18.3 mm
- net Net-(U1-X_1): track 14.0 -> 15.6 mm
- net /DATA3: track 15.1 -> 14.5 mm
- net /DATA0: track 8.13 -> 8.64 mm, vias 0 -> 1
- net /DATA1: track 13.7 -> 14.0 mm, vias 0 -> 1
Other:
- board size 42.3 x 28.3 mm -> 47.2 x 28.3 mm
