File: MXBreakout.kicad_sch (KiCad schematic)
At the start: 25 parts, among them U1 Wii-MX, Y1 32.768kHz

Commit message: Misc improvements to flex
Parts:
- renumbered C1 to C101, C2 to C102, C3 to C98, D1 to D31, R1 to R60
Changed lines of the file:
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@@
 (kicad_sch
-	(version 20240417)
+	(version 20250114)
 	(generator "eeschema")
-	(generator_version "8.99")
+	(generator_version "9.0")
 	(paper "A4")
 	(junction
@@
 	(label "SOFT"
 		(at 154.94 118.11 0)
-		(fields_autoplaced yes)
 		(effects
 			(font
@@
 	(label "DATA2"
 		(at 92.71 91.44 0)
-		(fields_autoplaced yes)
 		(effects
 			(font
@@
 	(label "DATA3"
 		(at 92.71 93.98 0)
-		(fields_autoplaced yes)
 		(effects
 			(font
@@
 	(label "POWER"
 		(at 154.94 107.95 0)
-		(fields_autoplaced yes)
 		(effects
 			(font
@@
 	(label "DATA0"
 		(at 92.71 86.36 0)
-		(fields_autoplaced yes)
 		(effects
 			(font
@@
 	(label "BATT"
 		(at 114.3 76.2 0)
-		(fields_autoplaced yes)
 		(effects
 			(font
@@
 	(label "DATA1"
 		(at 92.71 88.9 0)
-		(fields_autoplaced yes)
 		(effects
 			(font
@@
 	(label "RESET"
 		(at 154.94 97.79 0)
-		(fields_autoplaced yes)
 		(effects
 			(font
@@
 		(on_board yes)
 		(dnp no)
-		(property "Reference" "C2"
+		(property "Reference" "C102"
 			(at 39.3763 88.9 90)
 			(effects
@@
 			(project "MXBreakout"
 				(path "/b1683ed1-ed09-487c-8d86-af8ebf2f63f7"
-					(reference "C2")
+					(reference "C102")
 					(unit 1)
 				)
@@
 		(on_board yes)
 		(dnp no)
-		(property "Reference" "D1"
+		(property "Reference" "D31"
 			(at 96.52 69.85 0)
 			(effects
@@
 			(project "MXBreakout"
 				(path "/b1683ed1-ed09-487c-8d86-af8ebf2f63f7"
-					(reference "D1")
+					(reference "D31")
 					(unit 1)
 				)
@@
 		(dnp no)
 		(fields_autoplaced yes)
-		(property "Reference" "R1"
+		(property "Reference" "R60"
 			(at 104.14 71.12 90)
 			(effects
@@
 			(project "MXBreakout"
 				(path "/b1683ed1-ed09-487c-8d86-af8ebf2f63f7"
-					(reference "R1")
+					(reference "R60")
 					(unit 1)
 				)
@@
 		(dnp no)
 		(fields_autoplaced yes)
-		(property "Reference" "C3"
+		(property "Reference" "C98"
 			(at 96.52 120.6436 0)
 			(effects
@@
 			(project "MXBreakout"
 				(path "/b1683ed1-ed09-487c-8d86-af8ebf2f63f7"
-					(reference "C3")
+					(reference "C98")
 					(unit 1)
 				)
@@
 		(dnp no)
 		(fields_autoplaced yes)
-		(property "Reference" "C1"
+		(property "Reference" "C101"
 			(at 39.3763 68.58 90)
 			(effects
@@
 			(project "MXBreakout"
 				(path "/b1683ed1-ed09-487c-8d86-af8ebf2f63f7"
-					(reference "C1")
+					(reference "C101")
 					(unit 1)
 				)
@@
 		)
 	)
+	(embedded_fonts no)
 )
